Commit message: Fix ydlidar package

File: ros/workspace/src/medbot_description/urdf/medbot.urdf.xacro (robot description, xacro)
@@ -43,6 +43,6 @@
     <parent link="base_link"/>
     <child link="laser_frame"/>
-    <!-- Position LiDAR (e.g. 15cm forward, 10cm above chassis) -->
-    <origin xyz="0.15 0.0 0.12" rpy="0 0 0"/>
+    <!-- Position LiDAR in the center of the robot chassis -->
+    <origin xyz="0.0 0.0 0.10" rpy="0 0 0"/>
   </joint>
 </robot>

Commit message: Fix lidar position and ignore range in robot

File: ros/workspace/src/medbot_description/urdf/medbot.urdf.xacro (robot description, xacro)
@@ -3,9 +3,9 @@
   <!-- Base Footprint (Ground Projection) -->
   <link name="base_footprint"/>
-  <!-- Base Link (Chassis Center) -->
+  <!-- Base Link (Chassis Center: Length 44cm x Width 34cm) -->
   <link name="base_link">
     <visual>
       <geometry>
-        <box size="0.45 0.35 0.15"/>
+        <box size="0.44 0.34 0.15"/>
       </geometry>
       <material name="blue">
@@ -15,5 +15,5 @@
     <collision>
       <geometry>
-        <box size="0.45 0.35 0.15"/>
+        <box size="0.44 0.34 0.15"/>
       </geometry>
     </collision>
